Commit message: feat: New world, new robot and yaml file updated New world - Warehouse New robot - Size chnaged to fit in warehouse yaml file updated to describe the new warehouse map

File: my_robot/urdf/my_robot.xacro (robot description, xacro)
@@ -22,5 +22,5 @@
 			<origin xyz="0.0 0 0" rpy="0 0 0"/>
 			<geometry>
-				<box size=".4 .2 .1"/>
+				<box size=".2 .15 .07"/>
 			</geometry>
 		</collision>
@@ -28,29 +28,29 @@
 			<origin xyz="0.0 0 0" rpy="0 0 0"/>
 			<geometry>
-				<box size=".4 .2 .1"/>
+				<box size=".2 .15 .07"/>
 			</geometry>
 		</visual>
 		<collision name="back_caster_collision">
-			<origin xyz="-0.15 0 -0.05" rpy="0 0 0"/>
+			<origin xyz="-0.06 0 -0.02" rpy="0 0 0"/>
 			<geometry>
-				<sphere radius="0.0499"/>
+				<sphere radius="0.0299"/>
 			</geometry>
 		</collision>
 		<visual name="back_caster_visual">
-			<origin xyz="-0.15 0 -0.05" rpy="0 0 0"/>
+			<origin xyz="-0.06 0 -0.02" rpy="0 0 0"/>
 			<geometry>
-				<sphere radius="0.05"/>
+				<sphere radius="0.03"/>
 			</geometry>
 		</visual>
 		<collision name="front_caster_collision">
-			<origin xyz="0.15 0 -0.05" rpy="0 0 0"/>
+			<origin xyz="0.06 0 -0.02" rpy="0 0 0"/>
 			<geometry>
-				<sphere radius="0.0499"/>
+				<sphere radius="0.0299"/>
 			</geometry>
 		</collision>
 		<visual name="front_caster_visual">
-			<origin xyz="0.15 0 -0.05" rpy="0 0 0"/>
+			<origin xyz="0.06 0 -0.02" rpy="0 0 0"/>
 			<geometry>
-				<sphere radius="0.05"/>
+				<sphere radius="0.03"/>
 			</geometry>
 		</visual>
@@ -70,5 +70,5 @@
 			<origin xyz="0 0 0" rpy="0 1.5707 1.5707"/>
 			<geometry>
-				<cylinder radius="0.0999" length="0.0499"/>
+				<cylinder radius="0.0499" length="0.02499"/>
 			</geometry>
 		</collision>
@@ -76,5 +76,5 @@
 			<origin xyz="0 0 0" rpy="0 1.5707 1.5707"/>
 			<geometry>
-				<cylinder radius="0.1" length="0.05"/>
+				<cylinder radius="0.05" length="0.025"/>
 			</geometry>
 		</visual>
@@ -94,5 +94,5 @@
 			<origin xyz="0 0 0" rpy="0 1.5707 1.5707"/>
 			<geometry>
-				<cylinder radius="0.0999" length="0.0499"/>
+				<cylinder radius="0.0499" length="0.02499"/>
 			</geometry>
 		</collision>
@@ -100,10 +100,10 @@
 			<origin xyz="0 0 0" rpy="0 1.5707 1.5707"/>
 			<geometry>
-				<cylinder radius="0.1" length="0.05"/>
+				<cylinder radius="0.05" length="0.025"/>
 			</geometry>
 		</visual>
 	</link>
 	<joint name="left_wheel_hinge" type="continuous">
-		<origin xyz="0 0.15 0" rpy="0 0 0"/>
+		<origin xyz="0 0.088 0" rpy="0 0 0"/>
 		<child link="left_wheel"/>
 		<parent link="chassis"/>
@@ -113,5 +113,5 @@
 	</joint>
 	<joint name="right_wheel_hinge" type="continuous">
-		<origin xyz="0 -0.15 0" rpy="0 0 0"/>
+		<origin xyz="0 -0.088 0" rpy="0 0 0"/>
 		<child link="right_wheel"/>
 		<parent link="chassis"/>
@@ -145,5 +145,5 @@
 	</link>
 	<joint name="camera_joint" type="fixed">
-		<origin xyz="0.2 0 0" rpy="0 0 0"/>
+		<origin xyz="0.08 0 0" rpy="0 0 0"/>
 		<axis xyz="0 1 0" rpy="0 0 0"/>
 		<child link="camera"/>
@@ -177,5 +177,5 @@
 	</link>
 		<joint name="hokuyo_joint" type="fixed">
-			<origin xyz="0.15 0 0.1" rpy="0 0 0"/>
+			<origin xyz="0.05 0 0.07" rpy="0 0 0"/>
 			<axis xyz="0 1 0" rpy="0 0 0"/>
 			<child link="hokuyo"/>

Commit message: action: Map and Laser scan working Syntax issue in map.yaml file sorted Laser scan topic name changed in robot.gazebo. Remap still does not seems to work

File: my_robot/urdf/my_robot.xacro (robot description, xacro)
@@ -124,5 +124,5 @@
 		<inertial>
 			<mass value="0.1"/>
-			<origin xyz="0 0 0" rpy="0 0 0"/>
+			<origin xyz="0.05 0.05 0.05" rpy="0 0 0"/>
 			<inertia
 				ixx="1e-6" ixy="0" ixz="0"
@@ -132,5 +132,5 @@
 		</inertial>
 		<collision name="camera_collision">
-			<origin xyz="0.05 0.05 0.05" rpy="0 0 0"/>
+			<origin xyz="0 0 0" rpy="0 0 0"/>
 			<geometry>
 				<box size="0.05 0.05 0.05"/>
@@ -150,11 +150,10 @@
 		<parent link="chassis"/>
 	</joint>
+	<!-- LIDAR = Hokuyo Sensor -->
 	<link name="hokuyo">
-		<pose>0 0 0 0 0 0</pose>
+		<!-- <pose>0 0 0 0 0 0</pose> -->
 		<inertial>
 			<mass value="1e-5"/>
-			<geometry>
-				<box size="0.1 0.1 0.1"/>
-			</geometry>
+			<origin xyz="0 0 0" rpy="0 0 0"/>
 			<inertia
 				ixx="1e-6" ixy="0" ixz="0"
@@ -182,3 +181,15 @@
 			<parent link="chassis"/>
 		</joint>
+	<gazebo reference="chassis">
+    <material>Gazebo/Blue</material>
+  </gazebo>
+  <gazebo reference="left_wheel">
+    <material>Gazebo/Black</material>
+  </gazebo>
+  <gazebo reference="right_wheel">
+    <material>Gazebo/Black</material>
+  </gazebo>
+  <gazebo reference="camera">
+    <material>Gazebo/Red</material>
+  </gazebo>
 </robot>
